Commit message: Removed world link.

File: ur5_gripper/description/urdf/ur5_gripper_robot.urdf.xacro (robot description, xacro)
@@ -27,11 +27,5 @@
   <!-- gripper -->
   <xacro:robotiq_arg2f_140 prefix=""/>
-  <link name="world" />
-  <xacro:kinect xyz="0 1.7 1.0" rpy="0 0.0 -1.5" parent_frame="world" />
-  <joint name="world_joint" type="fixed">
-    <parent link="world" />
-    <child link = "base_link" />
-    <origin xyz="0.0 0.0 1.1" rpy="0.0 0.0 0.0" />
-  </joint>
+  <xacro:kinect xyz="0 1.7 0.4" rpy="0 0.0 -1.5" parent_frame="base_link" />
   <!-- sensor -->
   <xacro:robotiq_ft300 parent="tool0" prefix="">

Commit message: Added back world link and world joint.

File: ur5_gripper/description/urdf/ur5_gripper_robot.urdf.xacro (robot description, xacro)
@@ -27,4 +27,9 @@
   <!-- gripper -->
   <xacro:robotiq_arg2f_140 prefix=""/>
+  <joint name="world_joint" type="fixed">
+    <parent link="world" />
+    <child link = "base_link" />
+    <origin xyz="0.0 0.0 1.1" rpy="0.0 0.0 0.0" />
+  </joint>
   <!--xacro:kinect xyz="0 1.7 0.4" rpy="0 0.0 -1.5" parent_frame="base_link" /-->
   <!-- sensor -->

Commit message: Changed kinect version.
Changed the kinect v1 with kinect v2. Added a second kinect to the world.
Changed sensors_3d.yaml in moveit_config to work with both kinects.
Occupancy map includes pointclouds from both kinects.

File: ur5_gripper/description/urdf/ur5_gripper_robot.urdf.xacro (robot description, xacro)
@@ -13,5 +13,5 @@
   <xacro:include filename="$(find robotiq_ft_sensor)/urdf/robotiq_ft300.urdf.xacro" />
   <!-- kinect with plugin-->
-  <xacro:include filename="$(find ur5_gripper)/description/urdf/kinect_plugin.urdf.xacro" />
+  <xacro:include filename="$(find common_sensors)/urdf/sensors/kinect2.urdf.xacro" />
   <xacro:include filename="$(find robotiq_2f_140_gripper_visualization)/urdf/robotiq140_plugin.xacro" />
   <!-- arm -->
@@ -28,5 +28,10 @@
   <xacro:robotiq_arg2f_140 prefix=""/>
   <link name="world" />
-  <xacro:kinect xyz="0 1.7 1.0" rpy="0 0.0 -1.5" parent_frame="world" />
+  <xacro:kinect2  parent="world" name="kinectv2_1" >
+    <origin xyz="0 1.7 1.0" rpy="0 0.0 -1.5" />
+  </xacro:kinect2>
+  <xacro:kinect2  parent="world" name="kinectv2_2" >
+    <origin xyz="0 0 0.7" rpy="0.0 0.0 1.5" />
+  </xacro:kinect2>
   <joint name="world_joint" type="fixed">
     <parent link="world" />

Commit message: Changes for new kinectv2 cameras.

File: ur5_gripper/description/urdf/ur5_gripper_robot.urdf.xacro (robot description, xacro)
@@ -29,8 +29,11 @@
   <link name="world" />
   <xacro:kinect2  parent="world" name="kinectv2_1" >
-    <origin xyz="0 1.7 1.0" rpy="0 0.0 -1.5" />
+    <origin xyz="1.5 0.6 1.0" rpy="0.0 0.30 3.0" />
   </xacro:kinect2>
   <xacro:kinect2  parent="world" name="kinectv2_2" >
-    <origin xyz="0 0 0.7" rpy="0.0 0.0 1.5" />
+    <origin xyz="-0.7 0 1.0" rpy="0 0.15 1.5" />
+  </xacro:kinect2>
+  <xacro:kinect2  parent="world" name="kinectv2_3" >
+    <origin xyz="1.4 0.0 1.6" rpy="0.0 0.8 2.70" />
   </xacro:kinect2>
   <joint name="world_joint" type="fixed">
